File: EjectionBuddy/sense.kicad_sch (KiCad schematic)
At the start: 7 parts, among them U2 INA199B2

Commit message: More work on the side-mcu, ongoing
Changed lines of the file:
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@@
 	(text "V_{out} = 0.1 * V_{in}"
 		(exclude_from_sim no)
-		(at 50.038 150.622 0)
+		(at 49.276 152.908 0)
 		(effects
 			(font
