File: EjectionBuddy/mount.kicad_sch (KiCad schematic)
At the start: 4 parts

Commit message: Finished! QR and instruction pending
Parts:
- H1, H2, H3, H4: footprint (none) -> HoleNoMask_M4:HoleNoMask_4.3mm_M4
Changed lines of the file:
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@@
 			)
 		)
-		(property "Footprint" ""
+		(property "Footprint" "HoleNoMask_M4:HoleNoMask_4.3mm_M4"
 			(at 25.4 63.5 0)
 			(effects
@@
 		(instances
 			(project "EjectionBuddy"
-				(path "/8eb0a75f-d01a-4f77-b089-39fac6868a70/5ef685fe-bc2c-46ca-aa8b-f5bab32531ba"
+				(path "/8eb0a75f-d01a-4f77-b089-39fac6868a70/dc6dc8d0-470f-4975-8c29-8cff8cdf32db"
 					(reference "H4")
 					(unit 1)
@@
 			)
 		)
-		(property "Footprint" ""
+		(property "Footprint" "HoleNoMask_M4:HoleNoMask_4.3mm_M4"
 			(at 25.4 25.4 0)
 			(effects
@@
 		)
 		(instances
-			(project ""
-				(path "/8eb0a75f-d01a-4f77-b089-39fac6868a70/5ef685fe-bc2c-46ca-aa8b-f5bab32531ba"
+			(project "EjectionBuddy"
+				(path "/8eb0a75f-d01a-4f77-b089-39fac6868a70/dc6dc8d0-470f-4975-8c29-8cff8cdf32db"
 					(reference "H1")
 					(unit 1)
@@
 			)
 		)
-		(property "Footprint" ""
+		(property "Footprint" "HoleNoMask_M4:HoleNoMask_4.3mm_M4"
 			(at 25.4 50.8 0)
 			(effects
@@
 		(instances
 			(project "EjectionBuddy"
-				(path "/8eb0a75f-d01a-4f77-b089-39fac6868a70/5ef685fe-bc2c-46ca-aa8b-f5bab32531ba"
+				(path "/8eb0a75f-d01a-4f77-b089-39fac6868a70/dc6dc8d0-470f-4975-8c29-8cff8cdf32db"
 					(reference "H3")
 					(unit 1)
@@
 			)
 		)
-		(property "Footprint" ""
+		(property "Footprint" "HoleNoMask_M4:HoleNoMask_4.3mm_M4"
 			(at 25.4 38.1 0)
 			(effects
@@
 		(instances
 			(project "EjectionBuddy"
-				(path "/8eb0a75f-d01a-4f77-b089-39fac6868a70/5ef685fe-bc2c-46ca-aa8b-f5bab32531ba"
+				(path "/8eb0a75f-d01a-4f77-b089-39fac6868a70/dc6dc8d0-470f-4975-8c29-8cff8cdf32db"
 					(reference "H2")
 					(unit 1)
