File: EjectionBuddy/baro.kicad_sch (KiCad schematic)
At the start: 3 parts, among them U12 BMP280

Commit message: Side-mcu stm -> attiny, with improvements here and there
Parts:
- renumbered C36 to C26, C37 to C27
Changed lines of the file:
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@@
 		(dnp no)
 		(fields_autoplaced yes)
-		(property "Reference" "C36"
+		(property "Reference" "C26"
 			(at 83.82 40.6399 0)
 			(effects
@@
 			(project "EjectionBuddy"
 				(path "/8eb0a75f-d01a-4f77-b089-39fac6868a70/cbdf36e0-fe80-492b-aa20-c811f119c320"
-					(reference "C36")
+					(reference "C26")
 					(unit 1)
 				)
@@
 		(dnp no)
 		(fields_autoplaced yes)
-		(property "Reference" "#PWR0140"
+		(property "Reference" "#PWR0143"
 			(at 58.42 74.93 0)
 			(effects
@@
 			(project "EjectionBuddy"
 				(path "/8eb0a75f-d01a-4f77-b089-39fac6868a70/cbdf36e0-fe80-492b-aa20-c811f119c320"
-					(reference "#PWR0140")
+					(reference "#PWR0143")
 					(unit 1)
 				)
@@
 		(dnp no)
 		(fields_autoplaced yes)
-		(property "Reference" "#PWR0142"
+		(property "Reference" "#PWR0140"
 			(at 72.39 39.37 0)
 			(effects
@@
 			(project "EjectionBuddy"
 				(path "/8eb0a75f-d01a-4f77-b089-39fac6868a70/cbdf36e0-fe80-492b-aa20-c811f119c320"
-					(reference "#PWR0142")
+					(reference "#PWR0140")
 					(unit 1)
 				)
@@
 		(dnp no)
 		(fields_autoplaced yes)
-		(property "Reference" "#PWR0141"
+		(property "Reference" "#PWR0144"
 			(at 69.85 74.93 0)
 			(effects
@@
 			(project "EjectionBuddy"
 				(path "/8eb0a75f-d01a-4f77-b089-39fac6868a70/cbdf36e0-fe80-492b-aa20-c811f119c320"
-					(reference "#PWR0141")
+					(reference "#PWR0144")
 					(unit 1)
 				)
@@
 		(dnp no)
 		(fields_autoplaced yes)
-		(property "Reference" "#PWR0143"
+		(property "Reference" "#PWR0141"
 			(at 80.01 53.34 0)
 			(effects
@@
 			(project "EjectionBuddy"
 				(path "/8eb0a75f-d01a-4f77-b089-39fac6868a70/cbdf36e0-fe80-492b-aa20-c811f119c320"
-					(reference "#PWR0143")
+					(reference "#PWR0141")
 					(unit 1)
 				)
@@
 		(dnp no)
 		(fields_autoplaced yes)
-		(property "Reference" "#PWR0144"
+		(property "Reference" "#PWR0142"
 			(at 92.71 53.34 0)
 			(effects
@@
 			(project "EjectionBuddy"
 				(path "/8eb0a75f-d01a-4f77-b089-39fac6868a70/cbdf36e0-fe80-492b-aa20-c811f119c320"
-					(reference "#PWR0144")
+					(reference "#PWR0142")
 					(unit 1)
 				)
@@
 		(dnp no)
 		(fields_autoplaced yes)
-		(property "Reference" "C37"
+		(property "Reference" "C27"
 			(at 96.52 40.6399 0)
 			(effects
@@
 			(project "EjectionBuddy"
 				(path "/8eb0a75f-d01a-4f77-b089-39fac6868a70/cbdf36e0-fe80-492b-aa20-c811f119c320"
-					(reference "C37")
-					(unit 1)
-				)
+					(reference "C27")
+					(unit 1)
+				)
