File: EjectionBuddy/detach_sense.kicad_sch (KiCad schematic)
At the start: 9 parts, among them U10 TLP291, U9 TLP291

Commit message: Side-mcu stm -> attiny, with improvements here and there
Parts:
- renumbered C22 to C21, R27 to R28, R28 to R29, R29 to R30, R30 to R31, R31 to R32, R32 to R33
Changed lines of the file:
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@@
 		(dnp no)
 		(fields_autoplaced yes)
-		(property "Reference" "R32"
+		(property "Reference" "R33"
 			(at 53.34 77.4699 0)
 			(effects
@@
 			(project "EjectionBuddy"
 				(path "/8eb0a75f-d01a-4f77-b089-39fac6868a70/9490ce1c-6902-4b62-9fad-3e1d3d5b07c6"
-					(reference "R32")
+					(reference "R33")
 					(unit 1)
 				)
@@
 		(dnp no)
 		(fields_autoplaced yes)
-		(property "Reference" "R29"
+		(property "Reference" "R30"
 			(at 100.33 40.64 90)
 			(effects
@@
 			(project "EjectionBuddy"
 				(path "/8eb0a75f-d01a-4f77-b089-39fac6868a70/9490ce1c-6902-4b62-9fad-3e1d3d5b07c6"
-					(reference "R29")
+					(reference "R30")
 					(unit 1)
 				)
@@
 		(dnp no)
 		(fields_autoplaced yes)
-		(property "Reference" "C22"
+		(property "Reference" "C21"
 			(at 110.49 52.0699 0)
 			(effects
@@
 			(project "EjectionBuddy"
 				(path "/8eb0a75f-d01a-4f77-b089-39fac6868a70/9490ce1c-6902-4b62-9fad-3e1d3d5b07c6"
-					(reference "C22")
+					(reference "C21")
 					(unit 1)
 				)
@@
 		(dnp no)
 		(fields_autoplaced yes)
-		(property "Reference" "R27"
+		(property "Reference" "R28"
 			(at 87.63 38.0999 0)
 			(effects
@@
 			(project "EjectionBuddy"
 				(path "/8eb0a75f-d01a-4f77-b089-39fac6868a70/9490ce1c-6902-4b62-9fad-3e1d3d5b07c6"
-					(reference "R27")
+					(reference "R28")
 					(unit 1)
 				)
@@
 		(dnp no)
 		(fields_autoplaced yes)
-		(property "Reference" "R28"
+		(property "Reference" "R29"
 			(at 44.45 40.64 90)
 			(effects
@@
 			(project "EjectionBuddy"
 				(path "/8eb0a75f-d01a-4f77-b089-39fac6868a70/9490ce1c-6902-4b62-9fad-3e1d3d5b07c6"
-					(reference "R28")
+					(reference "R29")
 					(unit 1)
 				)
@@
 		(dnp no)
 		(fields_autoplaced yes)
-		(property "Reference" "R30"
+		(property "Reference" "R31"
 			(at 53.34 52.0699 0)
 			(effects
@@
 			(project "EjectionBuddy"
 				(path "/8eb0a75f-d01a-4f77-b089-39fac6868a70/9490ce1c-6902-4b62-9fad-3e1d3d5b07c6"
-					(reference "R30")
+					(reference "R31")
 					(unit 1)
 				)
@@
 		(dnp no)
 		(fields_autoplaced yes)
-		(property "Reference" "#PWR0131"
+		(property "Reference" "#PWR0132"
 			(at 80.01 86.36 0)
 			(effects
@@
 			(project "EjectionBuddy"
 				(path "/8eb0a75f-d01a-4f77-b089-39fac6868a70/9490ce1c-6902-4b62-9fad-3e1d3d5b07c6"
-					(reference "#PWR0131")
+					(reference "#PWR0132")
 					(unit 1)
 				)
@@
 		(dnp no)
 		(fields_autoplaced yes)
-		(property "Reference" "R31"
+		(property "Reference" "R32"
 			(at 44.45 66.04 90)
 			(effects
@@
 			(project "EjectionBuddy"
 				(path "/8eb0a75f-d01a-4f77-b089-39fac6868a70/9490ce1c-6902-4b62-9fad-3e1d3d5b07c6"
-					(reference "R31")
+					(reference "R32")
 					(unit 1)
 				)
@@
 		(dnp no)
 		(fields_autoplaced yes)
-		(property "Reference" "#PWR0130"
+		(property "Reference" "#PWR0131"
 			(at 106.68 66.04 0)
 			(effects
@@
 			(project "EjectionBuddy"
 				(path "/8eb0a75f-d01a-4f77-b089-39fac6868a70/9490ce1c-6902-4b62-9fad-3e1d3d5b07c6"
-					(reference "#PWR0130")
+					(reference "#PWR0131")
 					(unit 1)
 				)
@@
 		(dnp no)
 		(fields_autoplaced yes)
-		(property "Reference" "#PWR0128"
+		(property "Reference" "#PWR0129"
 			(at 85.09 36.83 0)
 			(effects
@@
 			(project "EjectionBuddy"
 				(path "/8eb0a75f-d01a-4f77-b089-39fac6868a70/9490ce1c-6902-4b62-9fad-3e1d3d5b07c6"
-					(reference "#PWR0128")
+					(reference "#PWR0129")
 					(unit 1)
 				)
@@
 		(dnp no)
 		(fields_autoplaced yes)
-		(property "Reference" "#PWR0129"
+		(property "Reference" "#PWR0130"
 			(at 80.01 60.96 0)
 			(effects
@@
 			(project "EjectionBuddy"
 				(path "/8eb0a75f-d01a-4f77-b089-39fac6868a70/9490ce1c-6902-4b62-9fad-3e1d3d5b07c6"
-					(reference "#PWR0129")
-					(unit 1)
-				)
+					(reference "#PWR0130")
+					(unit 1)
+				)

Commit message: Prodection version hw1.0 finished, with tidy-ups and bug-fixes
Other:
- note added: "V_{A} - V_{K} should < 12V The upper limit is currently determined by the power rating of those current-limiting resistors (resistive loss dissipation) As for the lower limit, delta-V above 3.3V should suffice"
- note removed: "V_{A} - V_{K} < 12V This value is currently determined by the resistor's power rating (to dissipate the resistive loss)"
Changed lines of the file:
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@@
 	(rectangle
 		(start 15.24 15.24)
-		(end 137.16 99.06)
+		(end 137.16 110.49)
 		(stroke
 			(width 0)
@@
 		)
 	)
-	(text "V_{A} - V_{K} < 12V\nThis value is currently determined\nby the resistor's power rating (to\ndissipate the resistive loss)"
-		(exclude_from_sim no)
-		(at 92.456 87.376 0)
+	(text "V_{A} - V_{K} should < 12V\nThe upper limit is currently determined by the\npower rating of those current-limiting resistors\n(resistive loss dissipation)\n\nAs for the lower limit, delta-V above 3.3V should suffice"
+		(exclude_from_sim no)
+		(at 27.178 97.028 0)
 		(effects
 			(font
@@
 		(dnp no)
 		(fields_autoplaced yes)
-		(property "Reference" "#PWR0132"
+		(property "Reference" "#PWR0133"
 			(at 80.01 86.36 0)
 			(effects
@@
 			(project "EjectionBuddy"
 				(path "/8eb0a75f-d01a-4f77-b089-39fac6868a70/9490ce1c-6902-4b62-9fad-3e1d3d5b07c6"
-					(reference "#PWR0132")
+					(reference "#PWR0133")
 					(unit 1)
 				)
@@
 		(dnp no)
 		(fields_autoplaced yes)
-		(property "Reference" "#PWR0131"
+		(property "Reference" "#PWR0132"
 			(at 106.68 66.04 0)
 			(effects
@@
 		(property "Description" "Power symbol creates a global label with name \"GND\" , ground"
 			(at 106.68 59.69 0)
+			(effects
+				(font
+					(size 1.27 1.27)
+				)
+				(hide yes)
+			)
+		)
+		(pin "1"
+		)
+		(instances
+			(project "EjectionBuddy"
+				(path "/8eb0a75f-d01a-4f77-b089-39fac6868a70/9490ce1c-6902-4b62-9fad-3e1d3d5b07c6"
+					(reference "#PWR0132")
+					(unit 1)
+				)
+			)
+		)
+	)
+	(symbol
+		(lib_id "power:+3.3V")
+		(at 85.09 33.02 0)
+		(unit 1)
+		(exclude_from_sim no)
+		(in_bom yes)
+		(on_board yes)
+		(dnp no)
+		(fields_autoplaced yes)
+		(property "Reference" "#PWR0130"
+			(at 85.09 36.83 0)
+			(effects
+				(font
+					(size 1.27 1.27)
+				)
+				(hide yes)
+			)
+		)
+		(property "Value" "+3.3V"
+			(at 85.09 27.94 0)
+			(effects
+				(font
+					(size 1.27 1.27)
+				)
+			)
+		)
+		(property "Footprint" ""
+			(at 85.09 33.02 0)
+			(effects
+				(font
+					(size 1.27 1.27)
+				)
+				(hide yes)
+			)
+		)
+		(property "Datasheet" ""
+			(at 85.09 33.02 0)
+			(effects
+				(font
+					(size 1.27 1.27)
+				)
+				(hide yes)
+			)
+		)
+		(property "Description" "Power symbol creates a global label with name \"+3.3V\""
+			(at 85.09 33.02 0)
+			(effects
+				(font
+					(size 1.27 1.27)
+				)
+				(hide yes)
+			)
+		)
+		(pin "1"
+		)
+		(instances
+			(project "EjectionBuddy"
+				(path "/8eb0a75f-d01a-4f77-b089-39fac6868a70/9490ce1c-6902-4b62-9fad-3e1d3d5b07c6"
+					(reference "#PWR0130")
+					(unit 1)
+				)
+			)
+		)
+	)
+	(symbol
+		(lib_id "power:GND")
+		(at 80.01 54.61 0)
+		(unit 1)
+		(exclude_from_sim no)
+		(in_bom yes)
+		(on_board yes)
+		(dnp no)
+		(fields_autoplaced yes)
+		(property "Reference" "#PWR0131"
+			(at 80.01 60.96 0)
+			(effects
+				(font
+					(size 1.27 1.27)
+				)
+				(hide yes)
+			)
+		)
+		(property "Value" "GND"
+			(at 80.01 59.69 0)
+			(effects
+				(font
+					(size 1.27 1.27)
+				)
+			)
+		)
+		(property "Footprint" ""
+			(at 80.01 54.61 0)
+			(effects
+				(font
+					(size 1.27 1.27)
+				)
+				(hide yes)
+			)
+		)
+		(property "Datasheet" ""
+			(at 80.01 54.61 0)
+			(effects
+				(font
+					(size 1.27 1.27)
+				)
+				(hide yes)
+			)
+		)
+		(property "Description" "Power symbol creates a global label with name \"GND\" , ground"
+			(at 80.01 54.61 0)
 			(effects
 				(font
@@
 					(unit 1)
 				)
-			)
-		)
-	)
-	(symbol
-		(lib_id "power:+3.3V")
-		(at 85.09 33.02 0)
-		(unit 1)
-		(exclude_from_sim no)
-		(in_bom yes)
-		(on_board yes)
-		(dnp no)
-		(fields_autoplaced yes)
-		(property "Reference" "#PWR0129"
-			(at 85.09 36.83 0)
-			(effects
-				(font
-					(size 1.27 1.27)
-				)
-				(hide yes)
-			)
-		)
-		(property "Value" "+3.3V"
-			(at 85.09 27.94 0)
-			(effects
-				(font
-					(size 1.27 1.27)
-				)
-			)
-		)
-		(property "Footprint" ""
-			(at 85.09 33.02 0)
-			(effects
-				(font
-					(size 1.27 1.27)
-				)
-				(hide yes)
-			)
-		)
-		(property "Datasheet" ""
-			(at 85.09 33.02 0)
-			(effects
-				(font
-					(size 1.27 1.27)
-				)
-				(hide yes)
-			)
-		)
-		(property "Description" "Power symbol creates a global label with name \"+3.3V\""
-			(at 85.09 33.02 0)
-			(effects
-				(font
-					(size 1.27 1.27)
-				)
-				(hide yes)
-			)
-		)
-		(pin "1"
-		)
-		(instances
-			(project "EjectionBuddy"
-				(path "/8eb0a75f-d01a-4f77-b089-39fac6868a70/9490ce1c-6902-4b62-9fad-3e1d3d5b07c6"
-					(reference "#PWR0129")
-					(unit 1)
-				)
-			)
-		)
-	)
-	(symbol
-		(lib_id "power:GND")
-		(at 80.01 54.61 0)
-		(unit 1)
-		(exclude_from_sim no)
-		(in_bom yes)
-		(on_board yes)
-		(dnp no)
-		(fields_autoplaced yes)
-		(property "Reference" "#PWR0130"
-			(at 80.01 60.96 0)
-			(effects
-				(font
-					(size 1.27 1.27)
-				)
-				(hide yes)
-			)
-		)
-		(property "Value" "GND"
-			(at 80.01 59.69 0)
-			(effects
-				(font
-					(size 1.27 1.27)
-				)
-			)
-		)
-		(property "Footprint" ""
-			(at 80.01 54.61 0)
-			(effects
-				(font
-					(size 1.27 1.27)
-				)
-				(hide yes)
-			)
-		)
-		(property "Datasheet" ""
-			(at 80.01 54.61 0)
-			(effects
-				(font
-					(size 1.27 1.27)
-				)
-				(hide yes)
-			)
-		)
-		(property "Description" "Power symbol creates a global label with name \"GND\" , ground"
-			(at 80.01 54.61 0)
-			(effects
-				(font
-					(size 1.27 1.27)
-				)
-				(hide yes)
-			)
-		)
-		(pin "1"
-		)
-		(instances
-			(project "EjectionBuddy"
-				(path "/8eb0a75f-d01a-4f77-b089-39fac6868a70/9490ce1c-6902-4b62-9fad-3e1d3d5b07c6"
-					(reference "#PWR0130")
-					(unit 1)
-				)
