File: EjectionBuddy/power_sense.kicad_sch (KiCad schematic)
At the start: 7 parts, among them U2 INA199B2

Commit message: Finished! QR and instruction pending
Parts:
- removed U2: INA199B2, Package_TO_SOT_SMD:SOT-363_SC-70-6, symbol Amplifier_Current:INA199xxDCK
- added U1: INA186xxQDCK, Package_TO_SOT_SMD:SOT-363_SC-70-6, symbol INA186:INA186xxQDCK
- C2: value 1n -> 0.1u
- R1: renamed from R3; value R -> 0.015; footprint FirstAero:ESC_CurrentSense_R_2x1206 -> Resistor_SMD:R_0805_2012Metric
- renumbered R4 to R2, R5 to R3, R6 to R4
Connections:
- net +3.3V: now also U1.3 (V+)
- net GND: now also U1.1 (REF), U1.2 (GND)
- net VBAT: now also U1.4 (+)
- net VM: no longer C2.2, R1.2
- net at R2.1: now also U1.6
- new net VS: C2.2, R1.2, U1.5 (-)
Other:
- note added: "A3 at gain 100V/V"
- note added: "XXV max"
- note removed: "26V max"
- note removed: "B2 at gain 100V/V"
- moved on the sheet: C1, R1, R2, R3, R4

Commit message: Slight improvements on routing and schematic
Parts:
- R1: value 0.015 -> 0.05
Other:
- note added: "A3 at gain 25V/V"
- note added: "V_{out} = 0.1 * V_{in} V"
- note added: "V_{out} = 0.8 V per A"
- note removed: "A3 at gain 100V/V"
- note removed: "V_{out} = 0.1 * V_{in}"
- moved on the sheet: C1, C2, R1, R2, U1

Commit message: Side-mcu stm -> attiny, with improvements here and there
Parts:
- renumbered R3 to R1, R1 to R2, R2 to R3
Changed lines of the file:
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@@
 		(dnp no)
 		(fields_autoplaced yes)
-		(property "Reference" "#PWR05"
+		(property "Reference" "#PWR03"
 			(at 35.56 45.72 0)
 			(effects
@@
 			(project ""
 				(path "/8eb0a75f-d01a-4f77-b089-39fac6868a70/f6fb7fef-7ebd-43c3-9a4f-2fff08951b4c"
-					(reference "#PWR05")
+					(reference "#PWR03")
 					(unit 1)
 				)
@@
 		(dnp no)
 		(fields_autoplaced yes)
-		(property "Reference" "#PWR08"
+		(property "Reference" "#PWR07"
 			(at 71.12 76.2 0)
 			(effects
@@
 			(project "EjectionBuddy"
 				(path "/8eb0a75f-d01a-4f77-b089-39fac6868a70/f6fb7fef-7ebd-43c3-9a4f-2fff08951b4c"
-					(reference "#PWR08")
+					(reference "#PWR07")
 					(unit 1)
 				)
@@
 		(dnp no)
 		(fields_autoplaced yes)
-		(property "Reference" "R1"
+		(property "Reference" "R2"
 			(at 44.45 53.3399 0)
 			(effects
@@
 			(project "EjectionBuddy"
 				(path "/8eb0a75f-d01a-4f77-b089-39fac6868a70/f6fb7fef-7ebd-43c3-9a4f-2fff08951b4c"
-					(reference "R1")
+					(reference "R2")
 					(unit 1)
 				)
@@
 		(dnp no)
 		(fields_autoplaced yes)
-		(property "Reference" "#PWR04"
+		(property "Reference" "#PWR02"
 			(at 71.12 43.18 0)
 			(effects
@@
 			(project "EjectionBuddy"
 				(path "/8eb0a75f-d01a-4f77-b089-39fac6868a70/f6fb7fef-7ebd-43c3-9a4f-2fff08951b4c"
-					(reference "#PWR04")
+					(reference "#PWR02")
 					(unit 1)
 				)
@@
 		(dnp no)
 		(fields_autoplaced yes)
-		(property "Reference" "R3"
+		(property "Reference" "R1"
 			(at 156.21 40.6399 0)
 			(effects
@@
 			(project "EjectionBuddy"
 				(path "/8eb0a75f-d01a-4f77-b089-39fac6868a70/f6fb7fef-7ebd-43c3-9a4f-2fff08951b4c"
-					(reference "R3")
+					(reference "R1")
 					(unit 1)
 				)
@@
 		(dnp no)
 		(fields_autoplaced yes)
-		(property "Reference" "#PWR010"
+		(property "Reference" "#PWR01"
 			(at 153.67 39.37 0)
 			(effects
@@
 			(project "EjectionBuddy"
 				(path "/8eb0a75f-d01a-4f77-b089-39fac6868a70/f6fb7fef-7ebd-43c3-9a4f-2fff08951b4c"
-					(reference "#PWR010")
+					(reference "#PWR01")
 					(unit 1)
 				)
@@
 		(dnp no)
 		(fields_autoplaced yes)
-		(property "Reference" "#PWR09"
+		(property "Reference" "#PWR08"
 			(at 38.1 78.74 0)
 			(effects
@@
 			(project "EjectionBuddy"
 				(path "/8eb0a75f-d01a-4f77-b089-39fac6868a70/f6fb7fef-7ebd-43c3-9a4f-2fff08951b4c"
-					(reference "#PWR09")
+					(reference "#PWR08")
 					(unit 1)
 				)
@@
 		(dnp no)
 		(fields_autoplaced yes)
-		(property "Reference" "#PWR011"
+		(property "Reference" "#PWR06"
 			(at 153.67 67.31 0)
 			(effects
@@
 			(project "EjectionBuddy"
 				(path "/8eb0a75f-d01a-4f77-b089-39fac6868a70/f6fb7fef-7ebd-43c3-9a4f-2fff08951b4c"
-					(reference "#PWR011")
+					(reference "#PWR06")
 					(unit 1)
 				)
@@
 		(dnp no)
 		(fields_autoplaced yes)
-		(property "Reference" "#PWR06"
+		(property "Reference" "#PWR04"
 			(at 41.91 45.72 0)
 			(effects
@@
 			(project "EjectionBuddy"
 				(path "/8eb0a75f-d01a-4f77-b089-39fac6868a70/f6fb7fef-7ebd-43c3-9a4f-2fff08951b4c"
-					(reference "#PWR06")
+					(reference "#PWR04")
 					(unit 1)
 				)
@@
 		(dnp no)
 		(fields_autoplaced yes)
-		(property "Reference" "R2"
+		(property "Reference" "R3"
 			(at 88.9 48.26 90)
 			(effects
@@
 			(project "EjectionBuddy"
 				(path "/8eb0a75f-d01a-4f77-b089-39fac6868a70/f6fb7fef-7ebd-43c3-9a4f-2fff08951b4c"
-					(reference "R2")
+					(reference "R3")
 					(unit 1)
 				)
@@
 		(dnp no)
 		(fields_autoplaced yes)
-		(property "Reference" "#PWR07"
+		(property "Reference" "#PWR05"
 			(at 82.55 49.53 0)
 			(effects
@@
 			(project "EjectionBuddy"
 				(path "/8eb0a75f-d01a-4f77-b089-39fac6868a70/f6fb7fef-7ebd-43c3-9a4f-2fff08951b4c"
-					(reference "#PWR07")
-					(unit 1)
-				)
+					(reference "#PWR05")
+					(unit 1)
+				)

Commit message: Prodection version hw1.0 finished, with tidy-ups and bug-fixes
Parts:
- U1: value INA186xxQDCK -> INA186A1
Other:
- note added: "A1 at gain 25V/V"
- note removed: "A3 at gain 25V/V"
- moved on the sheet: R1, R4
Changed lines of the file:
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@@
 	(rectangle
 		(start 119.38 15.24)
-		(end 185.42 82.55)
+		(end 185.42 91.44)
 		(stroke
 			(width 0)
@@
 	(text "V_{out} = 0.1 * V_{in} V"
 		(exclude_from_sim no)
-		(at 153.67 73.152 0)
+		(at 153.67 76.962 0)
 		(effects
 			(font
@@
 		)
 	)
-	(text "A3 at gain 25V/V"
+	(text "A1 at gain 25V/V"
 		(exclude_from_sim no)
 		(at 77.47 62.738 0)
@@
 	)
 	(junction
-		(at 153.67 48.26)
+		(at 153.67 52.07)
 		(diameter 0)
 		(color 0 0 0 0)
@@
 	(wire
 		(pts
-			(xy 153.67 48.26) (xy 148.59 48.26)
+			(xy 153.67 52.07) (xy 148.59 52.07)
 		)
 		(stroke
@@
 	(wire
 		(pts
-			(xy 153.67 45.72) (xy 153.67 48.26)
+			(xy 153.67 49.53) (xy 153.67 52.07)
 		)
 		(stroke
@@
 	(wire
 		(pts
-			(xy 153.67 35.56) (xy 153.67 38.1)
+			(xy 153.67 39.37) (xy 153.67 41.91)
 		)
 		(stroke
@@
 	(wire
 		(pts
-			(xy 153.67 58.42) (xy 153.67 60.96)
+			(xy 153.67 62.23) (xy 153.67 64.77)
 		)
 		(stroke
@@
 	(wire
 		(pts
-			(xy 153.67 48.26) (xy 153.67 50.8)
+			(xy 153.67 52.07) (xy 153.67 54.61)
 		)
 		(stroke
@@
 	(hierarchical_label "SENS_V"
 		(shape input)
-		(at 148.59 48.26 180)
+		(at 148.59 52.07 180)
 		(effects
 			(font
@@
 			)
 		)
-		(property "Value" "INA186xxQDCK"
+		(property "Value" "INA186A1"
 			(at 77.47 59.944 0)
 			(effects
@@
 		(dnp no)
 		(fields_autoplaced yes)
-		(property "Reference" "#PWR02"
+		(property "Reference" "#PWR01"
 			(at 71.12 43.18 0)
 			(effects
@@
 			(project "EjectionBuddy"
 				(path "/8eb0a75f-d01a-4f77-b089-39fac6868a70/f6fb7fef-7ebd-43c3-9a4f-2fff08951b4c"
-					(reference "#PWR02")
+					(reference "#PWR01")
 					(unit 1)
 				)
@@
 	(symbol
 		(lib_id "Device:R")
-		(at 153.67 41.91 0)
+		(at 153.67 45.72 0)
 		(unit 1)
 		(exclude_from_sim no)
@@
 		(fields_autoplaced yes)
 		(property "Reference" "R1"
-			(at 156.21 40.6399 0)
+			(at 156.21 44.4499 0)
 			(effects
 				(font
@@
 		)
 		(property "Value" "91k"
-			(at 156.21 43.1799 0)
+			(at 156.21 46.9899 0)
 			(effects
 				(font
@@
 		)
 		(property "Footprint" "Resistor_SMD:R_0603_1608Metric"
-			(at 151.892 41.91 90)
+			(at 151.892 45.72 90)
 			(effects
 				(font
@@
 		)
 		(property "Datasheet" "~"
-			(at 153.67 41.91 0)
+			(at 153.67 45.72 0)
 			(effects
 				(font
@@
 		)
 		(property "Description" "Resistor"
-			(at 153.67 41.91 0)
+			(at 153.67 45.72 0)
 			(effects
 				(font
@@
 	(symbol
 		(lib_id "Device:R")
-		(at 153.67 54.61 0)
+		(at 153.67 58.42 0)
 		(unit 1)
 		(exclude_from_sim no)
@@
 		(fields_autoplaced yes)
 		(property "Reference" "R4"
-			(at 156.21 53.3399 0)
+			(at 156.21 57.1499 0)
 			(effects
 				(font
@@
 		)
 		(property "Value" "10k"
-			(at 156.21 55.8799 0)
+			(at 156.21 59.6899 0)
 			(effects
 				(font
@@
 		)
 		(property "Footprint" "Resistor_SMD:R_0603_1608Metric"
-			(at 151.892 54.61 90)
+			(at 151.892 58.42 90)
 			(effects
 				(font
@@
 		)
 		(property "Datasheet" "~"
-			(at 153.67 54.61 0)
+			(at 153.67 58.42 0)
 			(effects
 				(font
@@
 		)
 		(property "Description" "Resistor"
-			(at 153.67 54.61 0)
+			(at 153.67 58.42 0)
 			(effects
 				(font
@@
 	(symbol
 		(lib_id "power:VBUS")
-		(at 153.67 35.56 0)
+		(at 153.67 39.37 0)
 		(unit 1)
 		(exclude_from_sim no)
@@
 		(dnp no)
 		(fields_autoplaced yes)
-		(property "Reference" "#PWR01"
+		(property "Reference" "#PWR02"
+			(at 153.67 43.18 0)
+			(effects
+				(font
+					(size 1.27 1.27)
+				)
+				(hide yes)
+			)
+		)
+		(property "Value" "VM"
+			(at 153.67 34.29 0)
+			(effects
+				(font
+					(size 1.27 1.27)
+				)
+			)
+		)
+		(property "Footprint" ""
 			(at 153.67 39.37 0)
 			(effects
@@
 			)
 		)
-		(property "Value" "VM"
-			(at 153.67 30.48 0)
-			(effects
-				(font
-					(size 1.27 1.27)
-				)
-			)
-		)
-		(property "Footprint" ""
-			(at 153.67 35.56 0)
-			(effects
-				(font
-					(size 1.27 1.27)
-				)
-				(hide yes)
-			)
-		)
 		(property "Datasheet" ""
-			(at 153.67 35.56 0)
+			(at 153.67 39.37 0)
 			(effects
 				(font
@@
 		)
 		(property "Description" "Power symbol creates a global label with name \"VBUS\""
-			(at 153.67 35.56 0)
+			(at 153.67 39.37 0)
 			(effects
 				(font
@@
 			(project "EjectionBuddy"
 				(path "/8eb0a75f-d01a-4f77-b089-39fac6868a70/f6fb7fef-7ebd-43c3-9a4f-2fff08951b4c"
-					(reference "#PWR01")
+					(reference "#PWR02")
 					(unit 1)
 				)
@@
 	(symbol
 		(lib_id "power:GND")
-		(at 153.67 60.96 0)
+		(at 153.67 64.77 0)
 		(unit 1)
 		(exclude_from_sim no)
@@
 		(fields_autoplaced yes)
 		(property "Reference" "#PWR06"
-			(at 153.67 67.31 0)
+			(at 153.67 71.12 0)
 			(effects
 				(font
@@
 		)
 		(property "Value" "GND"
-			(at 153.67 66.04 0)
+			(at 153.67 69.85 0)
 			(effects
 				(font
@@
 		)
 		(property "Footprint" ""
-			(at 153.67 60.96 0)
+			(at 153.67 64.77 0)
 			(effects
 				(font
@@
 		)
 		(property "Datasheet" ""
-			(at 153.67 60.96 0)
+			(at 153.67 64.77 0)
 			(effects
 				(font
@@
 		)
 		(property "Description" "Power symbol creates a global label with name \"GND\" , ground"
-			(at 153.67 60.96 0)
-			(effects
-				(font
+			(at 153.67 64.77 0)
+			(effects
+				(font
