File: EjectionBuddy/switch.kicad_sch (KiCad schematic)
At the start: 24 parts, among them Q1 NCE55P04S, Q2 NCE55P04S, Q3 UMH3N, Q4 UMH3N, Q5 UMH3N

Commit message: More work on the side-mcu, ongoing
Parts:
- added D6, D7, D8: 1N4007, Diode_SMD:Nexperia_CFP3_SOD-123W, symbol Diode:1N4007
- added JP2, JP3, JP4: SolderJumper_2_Open, symbol Jumper:SolderJumper_2_Open
Connections:
- net GND: now also D6.2 (A), D7.2 (A), D8.2 (A)
- net SVO1: now also JP2.2 (B)
- net SVO2: now also JP3.2 (B)
- net SVO3: now also JP4.2 (B)
- new net: D7.1 (K), JP3.1 (A)
- new net: D6.1 (K), JP2.1 (A)
- new net: D8.1 (K), JP4.1 (A)
Other:
- note added: "Flyback protection"
- note added: "Put those close to their output terminals"

Commit message: Finished! QR and instruction pending
Parts:
- removed D5: D_Zener, symbol Device:D_Zener
- removed JP2, JP3, JP4: SolderJumper_2_Open, symbol Jumper:SolderJumper_2_Open
- added D8: D_Zener, Diode_SMD:D_SOD-523, symbol Device:D_Zener
- added unit 2 of Q4
- C14: renamed from C8; footprint (none) -> Capacitor_SMD:C_0603_1608Metric
- D2, D3, D4: footprint (none) -> Diode_SMD:D_SOD-523
- R10: renamed from R12; value R -> 15k; footprint (none) -> Resistor_SMD:R_0603_1608Metric
- R11: renamed from R13; footprint (none) -> Resistor_SMD:R_0603_1608Metric
- R12: renamed from R14; footprint (none) -> Resistor_SMD:R_0603_1608Metric
- R13: renamed from R15; footprint (none) -> Resistor_SMD:R_0603_1608Metric
- R14: renamed from R17; value R -> 15k; footprint (none) -> Resistor_SMD:R_0603_1608Metric
- R15: renamed from R19; value R -> 15k; footprint (none) -> Resistor_SMD:R_0603_1608Metric
- R16: renamed from R18; value R -> 15k; footprint (none) -> Resistor_SMD:R_0603_1608Metric
- R17: renamed from R20; footprint (none) -> Resistor_SMD:R_0603_1608Metric
- R18: renamed from R16; footprint (none) -> Resistor_SMD:R_0603_1608Metric
- R5: renamed from R7; value R -> 15k; footprint (none) -> Resistor_SMD:R_0603_1608Metric
- R6: renamed from R8; value R -> 15k; footprint (none) -> Resistor_SMD:R_0603_1608Metric
- R7: renamed from R9; value R -> 15k; footprint (none) -> Resistor_SMD:R_0603_1608Metric
- R8: renamed from R10; value R -> 15k; footprint (none) -> Resistor_SMD:R_0603_1608Metric
- R9: renamed from R11; value R -> 15k; footprint (none) -> Resistor_SMD:R_0603_1608Metric
- renumbered D6 to D5, D7 to D6, D8 to D7
Connections:
- net GND: now also Q4.3 (C2), Q4.4 (E2), Q4.5 (B2)
- net SVO1: now also D5.1 (K)
- net SVO2: now also D6.1 (K)
- net SVO3: now also D7.1 (K)
- net VS: now also D8.1 (K)
- net at Q2.4 (G2), R14.2, R16.1: now also D8.2 (A)
Other:
- note added: "Unused"
- moved on the sheet: D5, D6, D7

Commit message: Prodection version hw1.0 finished, with tidy-ups and bug-fixes
Parts:
- D2, D3, D4, D8: value D_Zener -> D_Zener7V5
Other:
- note added: "Default closed"
- note added: "Default open"
Changed lines of the file:
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@@
 		)
 	)
+	(text "Default open"
+		(exclude_from_sim no)
+		(at 75.946 87.376 0)
+		(effects
+			(font
+				(size 1.27 1.27)
+			)
+			(justify left)
+		)
+	)
 	(text "Unused"
 		(exclude_from_sim no)
@@
 	(text "Put those close to their output terminals\n"
 		(exclude_from_sim no)
-		(at 248.666 152.654 0)
+		(at 223.52 153.162 0)
 		(effects
 			(font
 				(size 1.27 1.27)
 			)
-			(justify right)
 		)
 	)
@@
 		)
 	)
+	(text "Default closed"
+		(exclude_from_sim no)
+		(at 117.856 182.626 0)
+		(effects
+			(font
+				(size 1.27 1.27)
+			)
+			(justify left)
+		)
+	)
 	(text "low-pass filter\nf_{c} at 15.9 Hz"
 		(exclude_from_sim no)
@@
 			(table_cell "SW_STATE"
 				(exclude_from_sim no)
-				(at 76.2 74.93 0)
+				(at 118.11 170.18 0)
 				(size 11.43 2.54)
 				(margins 0.9525 0.9525 0.9525 0.9525)
@@
 			(table_cell "OUTPUT"
 				(exclude_from_sim no)
-				(at 87.63 74.93 0)
+				(at 129.54 170.18 0)
 				(size 11.43 2.54)
 				(margins 0.9525 0.9525 0.9525 0.9525)
@@
 			(table_cell "HIGH"
 				(exclude_from_sim no)
-				(at 76.2 77.47 0)
+				(at 118.11 172.72 0)
 				(size 11.43 2.54)
 				(margins 0.9525 0.9525 0.9525 0.9525)
@@
 				)
 			)
-			(table_cell "V_{bat}"
+			(table_cell "floating"
 				(exclude_from_sim no)
-				(at 87.63 77.47 0)
+				(at 129.54 172.72 0)
 				(size 11.43 2.54)
 				(margins 0.9525 0.9525 0.9525 0.9525)
@@
 			(table_cell "LOW"
 				(exclude_from_sim no)
-				(at 76.2 80.01 0)
+				(at 118.11 175.26 0)
 				(size 11.43 2.54)
 				(margins 0.9525 0.9525 0.9525 0.9525)
@@
 				)
 			)
-			(table_cell "floating"
+			(table_cell "V_{bat}"
 				(exclude_from_sim no)
-				(at 87.63 80.01 0)
+				(at 129.54 175.26 0)
 				(size 11.43 2.54)
 				(margins 0.9525 0.9525 0.9525 0.9525)
@@
 			(table_cell "FLOAT"
 				(exclude_from_sim no)
-				(at 76.2 82.55 0)
+				(at 118.11 177.8 0)
 				(size 11.43 2.54)
 				(margins 0.9525 0.9525 0.9525 0.9525)
@@
 				)
 			)
-			(table_cell "floating"
+			(table_cell "V_{bat}"
 				(exclude_from_sim no)
-				(at 87.63 82.55 0)
+				(at 129.54 177.8 0)
 				(size 11.43 2.54)
 				(margins 0.9525 0.9525 0.9525 0.9525)
@@
 			(table_cell "SW_STATE"
 				(exclude_from_sim no)
-				(at 118.11 170.18 0)
+				(at 76.2 74.93 0)
 				(size 11.43 2.54)
 				(margins 0.9525 0.9525 0.9525 0.9525)
@@
 			(table_cell "OUTPUT"
 				(exclude_from_sim no)
-				(at 129.54 170.18 0)
+				(at 87.63 74.93 0)
 				(size 11.43 2.54)
 				(margins 0.9525 0.9525 0.9525 0.9525)
@@
 			(table_cell "HIGH"
 				(exclude_from_sim no)
-				(at 118.11 172.72 0)
+				(at 76.2 77.47 0)
 				(size 11.43 2.54)
 				(margins 0.9525 0.9525 0.9525 0.9525)
@@
 				)
 			)
-			(table_cell "floating"
+			(table_cell "V_{bat}"
 				(exclude_from_sim no)
-				(at 129.54 172.72 0)
+				(at 87.63 77.47 0)
 				(size 11.43 2.54)
 				(margins 0.9525 0.9525 0.9525 0.9525)
@@
 			(table_cell "LOW"
 				(exclude_from_sim no)
-				(at 118.11 175.26 0)
+				(at 76.2 80.01 0)
 				(size 11.43 2.54)
 				(margins 0.9525 0.9525 0.9525 0.9525)
@@
 				)
 			)
-			(table_cell "V_{bat}"
+			(table_cell "floating"
 				(exclude_from_sim no)
-				(at 129.54 175.26 0)
+				(at 87.63 80.01 0)
 				(size 11.43 2.54)
 				(margins 0.9525 0.9525 0.9525 0.9525)
@@
 			(table_cell "FLOAT"
 				(exclude_from_sim no)
-				(at 118.11 177.8 0)
+				(at 76.2 82.55 0)
 				(size 11.43 2.54)
 				(margins 0.9525 0.9525 0.9525 0.9525)
@@
 				)
 			)
-			(table_cell "V_{bat}"
+			(table_cell "floating"
 				(exclude_from_sim no)
-				(at 129.54 177.8 0)
+				(at 87.63 82.55 0)
 				(size 11.43 2.54)
 				(margins 0.9525 0.9525 0.9525 0.9525)
@@
 			)
 		)
-		(property "Value" "D_Zener"
+		(property "Value" "D_Zener7V5"
 			(at 148.59 46.9899 90)
 			(effects
@@
 			)
 		)
-		(property "Value" "D_Zener"
+		(property "Value" "D_Zener7V5"
 			(at 109.22 142.2399 90)
 			(effects
@@
 			)
 		)
-		(property "Value" "D_Zener"
+		(property "Value" "D_Zener7V5"
 			(at 231.14 46.9899 90)
 			(effects
@@
 			)
 		)
-		(property "Value" "D_Zener"
+		(property "Value" "D_Zener7V5"
 			(at 67.31 46.9899 90)
 			(effects
